File: Snail_v1.kicad_sch (KiCad schematic)
At the start: 29 parts, among them J1 PWM_Connector, J5 Conn_ARM_SWD_TagConnect_TC203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, U1 STM32G431K6Tx

Commit message: Added layout
Parts:
- removed TP6: TestPoint, TestPoint:TestPoint_Pad_D2.5mm, symbol Connector:TestPoint
- added R23: 10kR, Resistor_SMD:R_0805_2012Metric_Pad1.20x1.40mm_HandSolder, symbol Device:R
- C22: footprint KiCad:830059539 -> 830059539:830059539
- TP1, TP2, TP3, TP4, TP5: footprint TestPoint:TestPoint_Pad_D2.5mm -> TestPoint:TestPoint_Pad_D1.0mm
Connections:
- net GND: now also R23.2
- net LED0: now also U1.6 (PA1)
- net LED1: now also U1.7 (PA2)
- net LED2: now also U1.20 (PA10)
- net DAC: now reaches R1.1
- net DAC: now also U1.9 (PA4)
- net at U1.31 (PB8): now also R23.1
- net USB_PWR_nINT: now reaches U1.5 (PA0)
- removed net SPI?_MISO: TP1.1, TP2.1, TP3.1, TP4.1, TP5.1, U1.10 (PA5), U1.11 (PA6), U1.12 (PA7), U1.13 (PB0), U1.25 (PA15), U1.26 (PB3), U1.27 (PB4), U1.28 (PB5), U1.29 (PB6), U1.30 (PB7), U1.7 (PA2), U1.8 (PA3), U1.9 (PA4)
- new net SPI1_MISO: TP5.1, U1.11 (PA6)
- new net SPI1_MOSI: TP4.1, U1.12 (PA7), U1.8 (PA3)
- new net SPI1_SCK: TP3.1, U1.10 (PA5)
- new net SPI1_nCS: U1.13 (PB0)
- new net UART?_Rx: TP2.1, U1.29 (PB6)
- new net UART?_Tx: TP1.1, U1.30 (PB7)
- new net USB_PWR_OUT1: U1.25 (PA15)
- new net USB_PWR_OUT2: U1.26 (PB3)
- no-connect marks 1 -> 2
